File: circuit/watchKiCad.kicad_pcb (KiCad board)
At the start: 2 copper layers, 20 parts, among them SW1 Button A, SW2 Button B, U1 LD1117S33TR_SOT223, U2 ATtiny84A-SSU, U3 SN74HC595D, U4 SN74HC595D, U5 KWM-20882CVB, Y1 4MHz

Commit message: Finished PCB
Parts:
- added REF**: SolderWire-0.1sqmm_1x01_D0.4mm_OD1mm, Connector_Wire:SolderWire-0.1sqmm_1x01_D0.4mm_OD1mm, F.Cu at (128.2, 114.0)
- added REF**: SolderWire-0.1sqmm_1x01_D0.4mm_OD1mm, Connector_Wire:SolderWire-0.1sqmm_1x01_D0.4mm_OD1mm, F.Cu at (128.2, 116.6)
- added REF**: SolderWire-0.1sqmm_1x01_D0.4mm_OD1mm, Connector_Wire:SolderWire-0.1sqmm_1x01_D0.4mm_OD1mm, F.Cu at (128.2, 119.2)
- added REF**: SolderWire-0.1sqmm_1x01_D0.4mm_OD1mm, Connector_Wire:SolderWire-0.1sqmm_1x01_D0.4mm_OD1mm, F.Cu at (128.2, 121.8)
- moved R10 60.6 mm to (149.6, 111.7), turned to 180 degrees
- moved R9 60.6 mm to (149.6, 109.2), turned to 180 degrees
- moved R5 58.2 mm to (141.3, 99.2)
- moved U3 55.8 mm to (142.7, 108.2)
- moved R3 55.8 mm to (141.3, 94.2), turned to 0 degrees
- moved R6 55.8 mm to (141.3, 101.7)
- moved SW1 55.8 mm to (143.7, 115.2)
- moved SW2 55.8 mm to (146.9, 121.7)
- moved U2 55.8 mm to (131.5, 106.2)
- moved U5 55.8 mm to (137.9, 94.2)
- moved Y1 55.8 mm to (132.4, 119.7)
- moved R2 55.8 mm to (154.2, 115.8)
- moved U1 55.8 mm to (131.7, 97.0)
- moved C1 55.8 mm to (136.4, 121.7)
- moved C2 55.8 mm to (136.4, 118.4)
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Connections:
- U2 pad 5: Net-(R2-Pad1) -> Net-(R1-Pad1)
- U2 pad 6: Net-(R1-Pad1) -> Net-(R2-Pad1)
- U3 pad 1: Net-(R3-Pad1) -> Net-(U3-Pad1)
- U3 pad 15: Net-(R10-Pad1) -> Net-(R7-Pad2)
- U3 pad 2: Net-(R5-Pad1) -> Net-(R8-Pad2)
- U3 pad 3: Net-(R6-Pad1) -> Net-(U3-Pad3)
- U3 pad 4: Net-(U3-Pad4) -> Net-(R9-Pad2)
- U3 pad 6: Net-(U3-Pad6) -> Net-(R10-Pad2)
- U4 pad 1: Net-(R7-Pad1) -> Net-(U4-Pad1)
- U4 pad 15: Net-(R4-Pad2) -> Net-(R6-Pad1)
- U4 pad 2: Net-(R8-Pad1) -> Net-(R5-Pad1)
- U4 pad 3: Net-(R9-Pad1) -> Net-(U4-Pad3)
- U4 pad 4: Net-(U4-Pad4) -> Net-(R4-Pad2)
- U4 pad 6: Net-(U4-Pad6) -> Net-(R3-Pad2)
- U5 pad 1: Net-(R3-Pad2) -> Net-(R3-Pad1)
- U5 pad 10: Net-(R8-Pad2) -> Net-(R9-Pad1)
- U5 pad 11: Net-(R10-Pad2) -> Net-(R8-Pad1)
- U5 pad 12: Net-(R9-Pad2) -> Net-(R7-Pad1)
- U5 pad 13: Net-(U4-Pad4) -> Net-(U4-Pad1)
- U5 pad 14: Net-(U4-Pad5) -> Net-(U4-Pad3)
- U5 pad 15: Net-(U4-Pad6) -> Net-(U4-Pad5)
- U5 pad 2: Net-(R5-Pad2) -> Net-(R4-Pad1)
- U5 pad 3: Net-(R4-Pad1) -> Net-(R5-Pad2)
- U5 pad 5: Net-(U3-Pad4) -> Net-(U3-Pad1)
- U5 pad 6: Net-(U3-Pad5) -> Net-(U3-Pad3)
- U5 pad 7: Net-(U3-Pad6) -> Net-(U3-Pad5)
- U5 pad 9: Net-(R7-Pad2) -> Net-(R10-Pad1)
Routing:
- net Net-(R1-Pad2): track 46.0 -> 104.8 mm
- net Net-(U2-Pad10): track 20.7 -> 49.0 mm
- net Net-(U2-Pad4): track 0.00 -> 24.9 mm, vias 0 -> 1
- net Net-(U2-Pad9): track 0.00 -> 15.9 mm, vias 0 -> 1
- net Net-(U2-Pad11): track 29.0 -> 42.4 mm
- net GND: track 93.0 -> 106.0 mm, vias 0 -> 4
- net Net-(U2-Pad12): track 24.4 -> 11.8 mm
- net Net-(U2-Pad7): track 0.00 -> 12.0 mm, vias 0 -> 1
- net Net-(U2-Pad8): track 0.00 -> 12.0 mm, vias 0 -> 1
- net Net-(R10-Pad1): track 13.0 -> 1.95 mm
- net Net-(U2-Pad13): track 26.8 -> 16.2 mm
- net Net-(R7-Pad1): track 10.6 -> 1.95 mm
- net Net-(R3-Pad1): track 10.4 -> 1.95 mm
- net Net-(R8-Pad1): track 10.4 -> 1.95 mm
- net Net-(R10-Pad2): track 1.95 -> 9.48 mm
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- added copper zone on B.Cu, net GND
- added copper zone on B.Cu, net VCC
Other:
- rule via_min_size: 0.4 -> 0.45
